File: output/pcbs/type-boy-40.kicad_pcb (KiCad board)
At the start: 2 copper layers, 242.4 x 71.3 mm, 165 parts

Commit message: Moved TypePak to left side.
Parts:
- removed the ? at (310.8, 142.9)
- removed the ? at (328.8, 154.5)
- removed the ? at (326.2, 142.9)
- removed B1: , E73:SW_TACT_ALPS_SKQGABE010
- removed the REF** at (322.0, 174.5)
- removed T1: , E73:SPDT_C128955
- removed XX5: , Untitled
- added ? (x2): , vik-logo-small, F.Cu at (68.5, 157.5)
- added ?: , SW_Tactile_SPST_Angled_PTS645Vx39-2LFS, F.Cu at (87.6, 206.8)
- added ?: , SW_CuK_OS102011MA1QN1_SPDT_Angled, F.Cu at (73.4, 207.1)
- added ?: , C_0805_2012Metric_Pad1.18x1.45mm_HandSolder, B.Cu at (73.2, 142.9)
- added ?: , C_0805_2012Metric_Pad1.18x1.45mm_HandSolder, B.Cu at (89.2, 142.9)
- added REF**: SolderJumper-2_P1.3mm_Open_RoundedPad1.0x1.5mm, Jumper:SolderJumper-2_P1.3mm_Open_RoundedPad1.0x1.5mm, B.Cu at (86.2, 160.2)
- added TH1: , vik-keyboard-throughole, F.Cu at (76.5, 157.5)
- added VIK OUT: , vik-keyboard-connector-horizontal, B.Cu at (77.5, 191.5)
- added XX1: , vik-keyboard-connector-horizontal, B.Cu at (75.5, 174.5)
- added XX3: , SolderJumper-3_default.3mm_Bridged12_RoundedPad1.0x1.5mm, B.Cu at (86.2, 155.0)
- added XX6: , Untitled, F.Cu at (68.5, 191.5)
- added XX8: , Untitled, B.Cu at (68.5, 191.5)
- XX4: footprint SolderJumper-3_default.3mm_Bridged12_RoundedPad1.0x1.5mm -> SolderJumper-2_from.3mm_Open_RoundedPad1.0x1.5mm
- moved _10 262.7 mm to (67.3, 206.6)
- moved _9 262.7 mm to (67.3, 142.4)
- moved ? 237.2 mm to (81.2, 137.5)
- moved ? 235.0 mm to (72.4, 143.0)
- moved ? 228.0 mm to (85.2, 174.5), turned to 90 degrees
- moved XX4 227.5 mm to (84.2, 197.8), turned to 180 degrees
- moved D1 16.0 mm to (108.0, 199.0)
- moved D10 16.0 mm to (144.0, 182.0)
- moved D11 16.0 mm to (144.0, 165.0)
- moved D12 16.0 mm to (144.0, 148.0)
- moved D13 16.0 mm to (162.0, 199.0)
- moved D14 16.0 mm to (162.0, 182.0)
- moved D15 16.0 mm to (162.0, 165.0)
- moved D16 16.0 mm to (162.0, 148.0)
- moved D17 16.0 mm to (180.0, 199.0)
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Connections:
- ? pad 10: row6 -> row3
- ? pad 11: row2 -> row7
- ? pad 12: row5 -> row4
- ? pad 13: row1 -> row8
- ? pad 6: row8 -> row1
- ? pad 7: row4 -> row5
- ? pad 8: row7 -> row2
- ? pad 9: row3 -> row6
- LED1 pad 2: LED37 -> LED48
- LED1 pad 4: LED36 -> LED47
- LED10 pad 2: LED34 -> LED27
- LED10 pad 4: LED33 -> LED26
- LED11 pad 2: LED15 -> LED22
- LED11 pad 4: LED14 -> LED21
- LED12 pad 2: LED10 -> LED3
- LED12 pad 4: LED9 -> LED2
- LED13 pad 2: LED40 -> LED45
- LED13 pad 4: LED39 -> LED44
- LED14 pad 2: LED33 -> LED28
- LED14 pad 4: LED32 -> LED27
- LED15 pad 2: LED16 -> LED21
- LED15 pad 4: LED15 -> LED20
- LED16 pad 2: LED9 -> LED4
- LED16 pad 4: LED8 -> LED3
- LED17 pad 2: LED41 -> LED44
- LED17 pad 4: LED40 -> LED43
- LED18 pad 2: LED32 -> LED29
- LED18 pad 4: LED31 -> LED28
- LED19 pad 2: LED17 -> LED20
- LED19 pad 4: LED16 -> LED19
- LED2 pad 2: LED36 -> LED25
- LED2 pad 4: LED35 -> LED24
- LED20 pad 2: LED8 -> LED5
- LED20 pad 4: LED7 -> LED4
- LED21 pad 2: LED42 -> LED43
- LED21 pad 4: LED41 -> LED42
- LED22 pad 2: LED31 -> LED30
- LED22 pad 4: LED30 -> LED29
- LED23 pad 2: LED18 -> LED19
- LED23 pad 4: LED17 -> LED18
- LED24 pad 2: LED7 -> LED6
- LED24 pad 4: LED6 -> LED5
- LED25 pad 2: LED43 -> LED42
- LED25 pad 4: LED42 -> LED41
- LED26 pad 2: LED30 -> LED31
- LED26 pad 4: LED29 -> LED30
- LED27 pad 2: LED19 -> LED18
- LED27 pad 4: LED18 -> LED17
- LED28 pad 2: LED6 -> LED7
- LED28 pad 4: LED5 -> LED6
- LED29 pad 2: LED44 -> LED41
- LED29 pad 4: LED43 -> LED40
- LED3 pad 2: LED13 -> LED24
- LED3 pad 4: LED12 -> LED23
- LED30 pad 2: LED29 -> LED32
- LED30 pad 4: LED28 -> LED31
- LED31 pad 2: LED20 -> LED17
- LED31 pad 4: LED19 -> LED16
- LED32 pad 2: LED5 -> LED8
- LED32 pad 4: LED4 -> LED7
- LED33 pad 2: LED45 -> LED40
- LED33 pad 4: LED44 -> LED39
- LED34 pad 2: LED28 -> LED33
- LED34 pad 4: LED27 -> LED32
- LED35 pad 2: LED21 -> LED16
- LED35 pad 4: LED20 -> LED15
- LED36 pad 2: LED4 -> LED9
- LED36 pad 4: LED3 -> LED8
- LED37 pad 2: LED46 -> LED39
- LED37 pad 4: LED45 -> LED38
- LED38 pad 2: LED27 -> LED34
- LED38 pad 4: LED26 -> LED33
- LED39 pad 2: LED22 -> LED15
- LED39 pad 4: LED21 -> LED14
- LED4 pad 2: LED12 -> LED1
- LED4 pad 4: LED11 -> RGB_OUT
- LED40 pad 2: LED3 -> LED10
- LED40 pad 4: LED2 -> LED9
- LED41 pad 2: LED47 -> LED38
- LED41 pad 4: LED46 -> LED37
- LED42 pad 2: LED26 -> LED35
- LED42 pad 4: LED25 -> LED34
- LED43 pad 2: LED23 -> LED14
- LED43 pad 4: LED22 -> LED13
- LED44 pad 2: LED2 -> LED11
- LED44 pad 4: LED1 -> LED10
- LED45 pad 2: LED48 -> LED37
- LED45 pad 4: LED47 -> LED36
- LED46 pad 2: LED25 -> LED36
- LED46 pad 4: LED24 -> LED35
- LED47 pad 2: LED24 -> LED13
- LED47 pad 4: LED23 -> LED12
- LED48 pad 2: LED1 -> LED12
- LED48 pad 4: RGB_OUT -> LED11
- LED5 pad 2: LED38 -> LED47
- LED5 pad 4: LED37 -> LED46
- LED6 pad 2: LED35 -> LED26
- LED6 pad 4: LED34 -> LED25
- LED7 pad 2: LED14 -> LED23
- LED7 pad 4: LED13 -> LED22
- LED8 pad 2: LED11 -> LED2
- LED8 pad 4: LED10 -> LED1
- LED9 pad 2: LED39 -> LED46
- LED9 pad 4: LED38 -> LED45
- XX4 pad 1: V33_ALWAYS -> VBUS
- XX4 pad 2: V33_JUMPER -> VIK_VBUS
Routing:
- net row7: track 108.2 -> 251.8 mm
- net row8: track 116.0 -> 253.7 mm
- net row2: track 249.2 -> 113.2 mm
- net row1: track 244.8 -> 111.7 mm
- net row5: track 134.9 -> 238.2 mm
- net row6: track 121.5 -> 223.8 mm
- net row3: track 218.0 -> 129.7 mm
- net row4: track 228.1 -> 143.6 mm
- net LED48: track 31.3 -> 107.4 mm, vias 0 -> 2
- net DATMIN: track 10.5 -> 79.8 mm
- net VIK_VBUS: track 0.00 -> 67.2 mm
- net DATPLUS: track 11.9 -> 78.3 mm
- net BAT_OUT: track 21.9 -> 84.5 mm, vias 0 -> 1
- net VBAT: track 24.9 -> 82.7 mm, vias 0 -> 1
- net VBUS: track 58.2 -> 112.2 mm, vias 3 -> 5
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Other:
- board size 242.4 x 71.3 mm -> 243.1 x 71.3 mm
- board text added: "3v3"
- board text added: "Always"
- board text added: "LED"
- board text added: "Skip"
- board text added: "VBUS"
- board text added: "VIK"
- board text removed: "On"
